File: eagle/bumper.brd (EAGLE design)
At the start: 81.3 x 67 mm, 25 parts, among them Q1 BC547, Q2 BC547

Commit message: Add files via upload
Parts:
- C2: value 47u -> 330u
- moved C5 1.27 mm to (25.4, 8.89)
- moved C8 1.27 mm to (25.4, 39.4)
Routing:
- net N$15: track 0.00 -> 295.9 mm
Other:
- board text added: "+"
- board text added: "-"
- board text added: "Bumper4Nano"
- board text added: "ppet36"
