File: eagle/bumper.sch (EAGLE design)
At the start: 25 parts, among them Q1 BC547, Q2 BC547

Commit message: Add files via upload
Parts:
- C2: value 47u -> 330u
Changed lines of the file:
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@@
 <part name="GND6" library="supply1" deviceset="GND" device=""/>
 <part name="P+4" library="supply1" deviceset="VCC" device=""/>
-<part name="C2" library="rcl" deviceset="CPOL-EU" device="E2,5-6E" value="47u"/>
+<part name="C2" library="rcl" deviceset="CPOL-EU" device="E2,5-6E" value="330u"/>
 <part name="C3" library="rcl" deviceset="C-EU" device="050-024X044" value="10n"/>
 <part name="C4" library="rcl" deviceset="C-EU" device="050-035X075" value="1u"/>
